File: betaBoard/betaBoard.kicad_pcb (KiCad board)
At the start: 2 copper layers, 65 x 45 mm, 132 parts, among them J1 DNP, J2 USB_B_Micro, J3 DNP, J4 DNP, J5 DNP, J6 DNP, SW1 C26638, SW2 C26638, U1 AMS1117-3.3_SOT223, U2 W25Q128JVSS / FM25Q64-SOB-T-G, U3 RP2040, U4 LM358, U5 LM358, U6 LM358, U7 LM358, Y1 X322512MSB4SI

Commit message: add PDFs and production file update (no significant changes)
Parts:
- J2: value USB_B_Micro -> AMPHENOL_10103592-0001LF
Other:
- board text added: "Castellations produce 2 errors in DRC"
- board text added: "DJ8TK"

Commit message: final ordered R1.0 pcb
Parts:
- SW1, SW2: footprint betaBoard:C26638 -> betaBoard:TS-1187A-B-A-B
- U2: value W25Q128JVSS / FM25Q64-SOB-T-G -> W25Q128JVSIQ
- U4, U5, U6, U7: footprint Package_SO:SOIC-8_5.23x5.23mm_P1.27mm -> Package_SO:SOIC-8_3.9x4.9mm_P1.27mm
- moved D22 3.28 mm to (85.8, 69.3)
- moved J4 2.17 mm to (53.8, 82.4)
- moved SW1 2.13 mm to (54.3, 72.5), turned to 90 degrees
- moved SW2 1.87 mm to (76.3, 83.0), turned to 180 degrees
- moved C29 1.37 mm to (85.7, 56.4)
- moved R27 1.37 mm to (87.2, 56.4)
- moved R28 1.37 mm to (84.2, 56.4)
- moved C28 1.35 mm to (87.2, 53.1)
- moved R25 1.35 mm to (84.2, 53.1)
- moved R26 1.35 mm to (85.7, 53.1)
- moved C22 1.35 mm to (87.2, 84.0)
- moved C23 1.35 mm to (85.7, 87.4)
- moved R17 1.35 mm to (84.2, 84.0)
- moved R18 1.35 mm to (85.7, 84.0)
- moved R19 1.35 mm to (87.2, 87.4)
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Connections:
- U3 pad 28: unconnected-(U3-Pad28) -> /MCU/GP17
Routing:
- net VCC: track 149.6 -> 130.1 mm
- net GND: track 38.1 -> 30.2 mm, vias 161 -> 172
- net Net-(U3-RUN): track 9.30 -> 15.8 mm
- net +3V3: track 209.2 -> 214.1 mm
- net /MCU/UART0_RX: track 15.0 -> 18.0 mm
- net /MCU/UART0_TX: track 13.5 -> 16.1 mm
- net /MCU/ADC2: track 14.0 -> 15.5 mm
- net /MCU/ADC3: track 22.9 -> 24.3 mm
- net /particle_sensor_array2/Diodes: track 20.7 -> 21.9 mm
- net /particle_sensor_array3/Diodes: track 21.4 -> 22.5 mm
- net /particle_sensor_array/Diodes: track 19.1 -> 20.2 mm
- net /MCU/GP10: track 16.2 -> 17.3 mm
- net Net-(U6B--): track 11.9 -> 10.9 mm
- net Net-(R6-Pad1): track 5.04 -> 5.84 mm
- net Net-(C35-Pad2): track 6.00 -> 6.80 mm
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Other:
- board text added: "Boot Select"
- board text added: "Reset"
