File: betaBoard/betaBoard.kicad_sch (KiCad schematic)
At the start: 40 parts, among them J1 DNP, J2 USB_B_Micro, J3 DNP, J4 DNP, J5 DNP, J6 DNP, U1 AMS1117-3.3_SOT223

Commit message: add PDFs and production file update (no significant changes)
Parts:
- J2: value USB_B_Micro -> AMPHENOL_10103592-0001LF
Changed lines of the file:
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@@
     (in_bom yes) (on_board yes)
     (property "Reference" "J2" (id 0) (at 111.76 47.625 0))
-    (property "Value" "USB_B_Micro" (id 1) (at 111.76 50.165 0))
+    (property "Value" "AMPHENOL_10103592-0001LF" (id 1) (at 111.76 50.165 0))
     (property "Footprint" "betaBoard:AMPHENOL_10103592-0001LF" (id 2) (at 115.57 62.23 0)
       (effects (font (size 1.27 1.27)) hide)
@@
     )
     (path "/a09ce6cf-1c69-4031-a0db-c493bb500671"
-      (reference "J2") (unit 1) (value "USB_B_Micro") (footprint "betaBoard:AMPHENOL_10103592-0001LF")
+      (reference "J2") (unit 1) (value "AMPHENOL_10103592-0001LF") (footprint "betaBoard:AMPHENOL_10103592-0001LF")
     )
     (path "/7a4fa37f-e348-40eb-8e06-344081235cb0"

Commit message: final ordered R1.0 pcb
Connections:
- no-connect marks 1 -> 2
Other:
- sheet MCU ports: added GP17; removed none
- moved on the sheet: D19, J4, J5, R1
