File: betaBoard/frontend.kicad_sch (KiCad schematic)
At the start: 16 parts, among them U5 LM358

Commit message: final ordered R1.0 pcb
Parts:
- U5: footprint Package_SO:SOIC-8_5.23x5.23mm_P1.27mm -> Package_SO:SOIC-8_3.9x4.9mm_P1.27mm
