File: betaBoard/mcu.kicad_sch (KiCad schematic)
At the start: 27 parts, among them SW1 C26638, SW2 C26638, U2 W25Q128JVSS / FM25Q64-SOB-T-G, U3 RP2040, Y1 X322512MSB4SI

Commit message: final ordered R1.0 pcb
Parts:
- SW1, SW2: footprint betaBoard:C26638 -> betaBoard:TS-1187A-B-A-B
- U2: value W25Q128JVSS / FM25Q64-SOB-T-G -> W25Q128JVSIQ
Connections:
- net GP17: now reaches U3.28 (GPIO17)
- no-connect marks 19 -> 18
