File: hardware/betaBoard_r2.0/mcu.kicad_sch (KiCad schematic)
At the start: 27 parts, among them SW1 TS-1187A-B-A-B, SW2 TS-1187A-B-A-B, U2 W25Q128JVSIQ, U3 RP2040, Y1 X322512MSB4SI

Commit message: main r2.0 design done
Connections:
- net GP23: now reaches U3.35 (GPIO23)
- no-connect marks 18 -> 17
Other:
- moved on the sheet: C10, C11, C12, C13, C14, C15, C16, C17, C3, C4, C5, C6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
